File: keeb.kicad_pcb (KiCad board)
At the start: 2 copper layers, 161.9 x 116.3 mm, 70 parts

Commit message: add mounting holes
Parts:
- added REF**: MountingHole_3.2mm_M3_ISO7380, MountingHole:MountingHole_3.2mm_M3_ISO7380, F.Cu at (60.0, 22.5)
- added REF**: MountingHole_3.2mm_M3_ISO7380, MountingHole:MountingHole_3.2mm_M3_ISO7380, F.Cu at (134.0, 75.0)
- added REF**: MountingHole_3.2mm_M3_ISO7380, MountingHole:MountingHole_3.2mm_M3_ISO7380, F.Cu at (83.5, 24.5)
- added REF**: MountingHole_3.2mm_M3_ISO7380, MountingHole:MountingHole_3.2mm_M3_ISO7380, F.Cu at (38.0, 113.0)
- added REF**: MountingHole_3.2mm_M3_ISO7380, MountingHole:MountingHole_3.2mm_M3_ISO7380, F.Cu at (74.5, 90.5)
- added REF**: MountingHole_3.2mm_M3_ISO7380, MountingHole:MountingHole_3.2mm_M3_ISO7380, F.Cu at (121.0, 101.5)
- added REF**: MountingHole_3.2mm_M3_ISO7380, MountingHole:MountingHole_3.2mm_M3_ISO7380, F.Cu at (127.0, 51.5)
